File: Hardware/PCB.brd (EAGLE design)
At the start: 46 x 35 mm, 105 parts, among them IC1 BQ25180YBGR, IC2 DRV2605YZFR, IC3 BMA423_BMA423, IC9 RT6160AWSC_RT6160AWSC, J1 503480-2400, J2 TC2030-IDC_TC2030-IDCCABLU, J4 KH-TYPE-C-16P, Q1 20V/4.2A/52mΩ/1.4W, Q3 SI1308EDL-T1-GE3, U1 NRF52840_QF, U3 MAX17048G+T10, X1 32MHZ, X2\ 32.768kHz

Commit message: Add files via upload
Connections:
- removed net N$26: U1.P$74, U1.P$75, U1.P$76, U1.P$77, U1.P$78, U1.P$79, U1.P$80, U1.P$81, U1.P$82, U1.P$83, U1.P$84, U1.P$85, U1.P$86, U1.P$87, U1.P$88, U1.P$89, U1.P$90
- removed net N$7: D3.2
- removed net N.C.: C8.2
- net GND: now also C8.2, D3.2, U1.P$74, U1.P$75, U1.P$76, U1.P$77, U1.P$78, U1.P$79, U1.P$80, U1.P$81, U1.P$82, U1.P$83, U1.P$84, U1.P$85, U1.P$86, U1.P$87, U1.P$88, U1.P$89, U1.P$90
Routing:
- net N$26: track 26.7 -> 0.00 mm
- net GND: track 82.0 -> 108.7 mm
- net 3V3: track 134.2 -> 131.4 mm
- net RESET: track 35.3 -> 33.8 mm
