File: Hardware/Schematic.sch (EAGLE design)
At the start: 105 parts, among them IC1 BQ25180YBGR, IC2 DRV2605YZFR, IC3 BMA423_BMA423, IC9 RT6160AWSC_RT6160AWSC, J1 503480-2400, J2 TC2030-IDC_TC2030-IDCCABLU, J4 KH-TYPE-C-16P, Q1 20V/4.2A/52mΩ/1.4W, Q3 SI1308EDL-T1-GE3, U1 NRF52840_QF, U3 MAX17048G+T10, X1 32MHZ, X2\ 32.768kHz

Commit message: Add files via upload
Connections:
- removed net N$26: U1.VSS_PAD
- removed net N$7: D3.GND
- removed net N.C.: C8.2
- net GND: now also C8.2, D3.GND, U1.VSS_PAD
Changed lines of the file:
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@@
 <setting verticaltext="up"/>
 </settings>
-<grid distance="0.1" unitdist="inch" unit="inch" style="lines" multiple="1" display="no" altdistance="0.01" altunitdist="inch" altunit="inch"/>
+<grid distance="0.05" unitdist="inch" unit="inch" style="lines" multiple="1" display="no" altdistance="0.01" altunitdist="inch" altunit="inch"/>
 <layers>
 <layer number="1" name="Top" color="4" fill="1" visible="no" active="no"/>
@@
 <attribute name="VALUE" x="300.99" y="60.96" size="1.778" layer="96" align="bottom-center"/>
 </instance>
-<instance part="SUPPLY3" gate="G$1" x="307.34" y="99.06" smashed="yes">
-<attribute name="VALUE" x="307.34" y="96.52" size="1.778" layer="96" align="bottom-center"/>
+<instance part="SUPPLY3" gate="G$1" x="307.34" y="97.79" smashed="yes">
+<attribute name="VALUE" x="307.34" y="95.25" size="1.778" layer="96" align="bottom-center"/>
 </instance>
 <instance part="SUPPLY4" gate="G$1" x="287.02" y="124.46" smashed="yes">
@@
 <pinref part="C13" gate="C$1" pin="1"/>
 </segment>
+<segment>
+<wire x1="262.89" y1="106.68" x2="276.86" y2="106.68" width="0.1524" layer="91"/>
+<wire x1="276.86" y1="106.68" x2="276.86" y2="102.87" width="0.1524" layer="91"/>
+<pinref part="SUPPLY40" gate="G$1" pin="GND"/>
+<pinref part="U1" gate="G$1" pin="VSS_PAD"/>
+</segment>
+<segment>
+<wire x1="307.34" y1="105.41" x2="307.34" y2="100.33" width="0.1524" layer="91"/>
+<pinref part="SUPPLY3" gate="G$1" pin="GND"/>
+<pinref part="C8" gate="C$1" pin="2"/>
+</segment>
 </net>
 <net name="N$29" class="0">
@@
 <net name="N$35" class="0">
 <segment>
-<wire x1="119.38" y1="182.88" x2="119.38" y2="181.61" width="0.1524" layer="91"/>
 <wire x1="119.38" y1="181.61" x2="119.38" y2="177.8" width="0.1524" layer="91"/>
 <wire x1="184.15" y1="154.94" x2="130.81" y2="154.94" width="0.1524" layer="91"/>
@@
 </segment>
 </net>
-<net name="N$26" class="0">
-<segment>
-<wire x1="262.89" y1="106.68" x2="276.86" y2="106.68" width="0.1524" layer="91"/>
-<wire x1="276.86" y1="106.68" x2="276.86" y2="102.87" width="0.1524" layer="91"/>
-<pinref part="SUPPLY40" gate="G$1" pin="GND"/>
-<pinref part="U1" gate="G$1" pin="VSS_PAD"/>
-</segment>
-</net>
 <net name="VBUS" class="1">
 <segment>
 <wire x1="21.59" y1="232.41" x2="21.59" y2="236.22" width="0.1524" layer="91"/>
 <wire x1="21.59" y1="236.22" x2="49.53" y2="236.22" width="0.1524" layer="91"/>
-<wire x1="21.59" y1="236.22" x2="11.43" y2="236.22" width="0.1524" layer="91"/>
-<label x="11.43" y="236.22" size="1.27" layer="95" rot="R180" xref="yes"/>
-<junction x="21.59" y="236.22"/>
+<wire x1="21.59" y1="236.22" x2="16.51" y2="236.22" width="0.1524" layer="91"/>
+<label x="16.51" y="236.22" size="1.27" layer="95" rot="R180" xref="yes"/>
 <pinref part="IC1" gate="G$1" pin="IN"/>
 <pinref part="C38" gate="C$1" pin="1"/>
+<junction x="21.59" y="236.22"/>
 </segment>
 <segment>
@@
 <pinref part="U1" gate="G$1" pin="VDD@W1"/>
 <pinref part="U1" gate="G$1" pin="VDDH@Y2"/>
+<label x="162.56" y="124.46" size="1.27" layer="95" rot="R180" xref="yes"/>
 </segment>
 <segment>
@@
 <label x="271.78" y="124.46" size="1.27" layer="95" xref="yes"/>
 <pinref part="U1" gate="G$1" pin="P1.01@Y23"/>
-</segment>
-</net>
-<net name="N.C." class="0">
-<segment>
-<wire x1="307.34" y1="105.41" x2="307.34" y2="101.6" width="0.1524" layer="91"/>
-<pinref part="SUPPLY3" gate="G$1" pin="GND"/>
-<pinref part="C8" gate="C$1" pin="2"/>
 </segment>
 </net>
@@
 <pinref part="C42" gate="C$1" pin="2"/>
 </segment>
+<segment>
+<wire x1="311.15" y1="92.71" x2="304.8" y2="92.71" width="0.1524" layer="91"/>
+<wire x1="304.8" y1="92.71" x2="304.8" y2="86.36" width="0.1524" layer="91"/>
+<pinref part="SUPPLY59" gate="G$1" pin="GND"/>
+<pinref part="D3" gate="G$1" pin="GND"/>
+</segment>
 </net>
 <net name="N$6" class="0">
@@
 <wire x1="308.61" y1="173.99" x2="308.61" y2="171.45" width="0.1524" layer="91"/>
 <wire x1="308.61" y1="173.99" x2="342.9" y2="173.99" width="0.1524" layer="91"/>
-<wire x1="342.9" y1="173.99" x2="342.9" y2="171.45" width="0.1524" layer="91"/>
 <label x="345.44" y="173.99" size="1.27" layer="95" rot="MR180" xref="yes"/>
-<junction x="308.61" y="173.99"/>
 <pinref part="R5" gate="G$1" pin="2"/>
 <pinref part="R8" gate="G$1" pin="2"/>
 <pinref part="R7" gate="G$1" pin="2"/>
+<wire x1="342.9" y1="173.99" x2="342.9" y2="171.45" width="0.1524" layer="91"/>
+<wire x1="342.9" y1="173.99" x2="345.44" y2="173.99" width="0.1524" layer="91"/>
+<junction x="308.61" y="173.99"/>
+<junction x="342.9" y="173.99"/>
 </segment>
 <segment>
@@
 </segment>
 </net>
-<net name="N$7" class="0">
-<segment>
-<wire x1="311.15" y1="92.71" x2="304.8" y2="92.71" width="0.1524" layer="91"/>
-<wire x1="304.8" y1="92.71" x2="304.8" y2="86.36" width="0.1524" layer="91"/>
-<pinref part="SUPPLY59" gate="G$1" pin="GND"/>
-<pinref part="D3" gate="G$1" pin="GND"/>
-</segment>
-</net>
 <net name="D_N" class="0">
 <segment>
@@
 </sheet>
 </sheets>
+<errors>
+</errors>
 </schematic>
 </drawing>
